Commit message: expose more of robot_arm control rename pybullet_utils to avoid clash update franka_panda urdfs to match others

File: tactile_sim/assets/embodiment_assets/combined_urdfs/franka_panda_flat_tactip.urdf (robot description, URDF)
Before this commit: robot panda, 13 links, 12 joints
Links:
- link ee_link: geometry collision sphere radius=0.00100; visual sphere radius=0.00100
Joints:
- joint ee_joint: origin xyz=0.00000 0.00000 0.10700 rpy=0.00000 -0.00000 0.00000 -> xyz=0.00000 0.00000 0.10700 rpy=3.14000 -0.00000 1.57000
- joint joint_dummy1: origin xyz=0.00000 0.00000 0.00000 rpy=0.00000 0.00000 -1.57080 -> xyz=0.00000 0.00000 0.00000 rpy=-3.14159 0.00000 3.14159

File: tactile_sim/assets/embodiment_assets/combined_urdfs/franka_panda_mini_tactip.urdf (robot description, URDF)
Before this commit: robot panda, 13 links, 12 joints
Links:
- link ee_link: geometry collision sphere radius=0.00100; visual sphere radius=0.00100
Joints:
- joint ee_joint: origin xyz=0.00000 0.00000 0.10700 rpy=0.00000 -0.00000 0.00000 -> xyz=0.00000 0.00000 0.10700 rpy=3.14000 -0.00000 1.57000
- joint joint_dummy1: origin xyz=0.00000 0.00000 0.00000 rpy=0.00000 0.00000 -1.57080 -> xyz=0.00000 0.00000 0.00000 rpy=-3.14159 0.00000 3.14159

File: tactile_sim/assets/embodiment_assets/combined_urdfs/franka_panda_right_angle_digit.urdf (robot description, URDF)
Before this commit: robot panda, 13 links, 12 joints
Links:
- link ee_link: geometry collision sphere radius=0.00100; visual sphere radius=0.00100
Joints:
- joint ee_joint: origin xyz=0.00000 0.00000 0.10700 rpy=0.00000 -0.00000 0.00000 -> xyz=0.00000 0.00000 0.10700 rpy=3.14000 -0.00000 1.57000
- joint joint_dummy1: origin xyz=0.00000 0.00500 0.06000 rpy=0.00000 1.57080 3.14159 -> xyz=0.00000 0.00500 -0.06000 rpy=-1.57080 -1.57080 3.14159

File: tactile_sim/assets/embodiment_assets/combined_urdfs/franka_panda_right_angle_digitac.urdf (robot description, URDF)
Before this commit: robot panda, 13 links, 12 joints
Links:
- link ee_link: geometry collision sphere radius=0.00100; visual sphere radius=0.00100
Joints:
- joint ee_joint: origin xyz=0.00000 0.00000 0.10700 rpy=0.00000 -0.00000 0.00000 -> xyz=0.00000 0.00000 0.10700 rpy=3.14000 -0.00000 1.57000
- joint joint_dummy1: origin xyz=0.00000 0.00500 0.06000 rpy=0.00000 1.57080 3.14159 -> xyz=0.00000 0.00500 -0.06000 rpy=-1.57080 -1.57080 3.14159

File: tactile_sim/assets/embodiment_assets/combined_urdfs/franka_panda_right_angle_tactip.urdf (robot description, URDF)
Before this commit: robot panda, 14 links, 13 joints
Links:
- link ee_link: geometry collision sphere radius=0.00100; visual sphere radius=0.00100
Joints:
- joint ee_joint: origin xyz=0.00000 0.00000 0.10700 rpy=0.00000 -0.00000 0.00000 -> xyz=0.00000 0.00000 0.10700 rpy=3.14000 -0.00000 1.57000
- joint joint_dummy1: origin xyz=0.00000 0.00500 0.06000 rpy=0.00000 1.57080 3.14159 -> xyz=0.00000 0.00500 -0.06000 rpy=-1.57080 -1.57080 3.14159

File: tactile_sim/assets/embodiment_assets/combined_urdfs/franka_panda_standard_digit.urdf (robot description, URDF)
Before this commit: robot panda, 13 links, 12 joints
Links:
- link ee_link: geometry collision sphere radius=0.00100; visual sphere radius=0.00100
Joints:
- joint ee_joint: origin xyz=0.00000 0.00000 0.10700 rpy=0.00000 -0.00000 0.00000 -> xyz=0.00000 0.00000 0.10700 rpy=3.14000 -0.00000 1.57000
- joint joint_dummy1: origin xyz=0.00000 0.00000 0.00000 rpy=0.00000 0.00000 -1.57080 -> xyz=0.00000 0.00000 0.00000 rpy=-3.14159 0.00000 3.14159

File: tactile_sim/assets/embodiment_assets/combined_urdfs/franka_panda_standard_digitac.urdf (robot description, URDF)
Before this commit: robot panda, 13 links, 12 joints
Links:
- link ee_link: geometry collision sphere radius=0.00100; visual sphere radius=0.00100
Joints:
- joint ee_joint: origin xyz=0.00000 0.00000 0.10700 rpy=0.00000 -0.00000 0.00000 -> xyz=0.00000 0.00000 0.10700 rpy=3.14000 -0.00000 1.57000
- joint joint_dummy1: origin xyz=0.00000 0.00000 0.00000 rpy=0.00000 0.00000 -1.57080 -> xyz=0.00000 0.00000 0.00000 rpy=-3.14159 0.00000 3.14159

File: tactile_sim/assets/embodiment_assets/combined_urdfs/franka_panda_standard_tactip.urdf (robot description, URDF)
Before this commit: robot panda, 13 links, 12 joints
Links:
- link ee_link: geometry collision sphere radius=0.00100; visual sphere radius=0.00100
Joints:
- joint ee_joint: origin xyz=0.00000 0.00000 0.10700 rpy=0.00000 -0.00000 0.00000 -> xyz=0.00000 0.00000 0.10700 rpy=3.14000 -0.00000 1.57000
- joint joint_dummy1: origin xyz=0.00000 0.00000 0.00000 rpy=0.00000 0.00000 -1.57080 -> xyz=0.00000 0.00000 0.00000 rpy=-3.14159 0.00000 3.14159

File: tactile_sim/assets/robot_arm_assets/franka_panda/urdfs/franka_panda.urdf (robot description, URDF)
Before this commit: robot panda, 10 links, 9 joints
Links:
- link ee_link: geometry collision sphere radius=0.001; visual sphere radius=0.001
Joints:
- joint ee_joint: origin xyz=0 0 0.107 rpy=0.0 0.0 0.0 -> xyz=0.0 0.0 0.107 rpy=3.14 0.0 1.57
