Commit message: tidy assets, sort reference images combine_urdfs script now creates clean urdfs

File: tactile_sim/assets/embodiment_assets/combined_urdfs/cr3_flat_tactip.urdf (robot description, URDF)
Before this commit: robot cr3_robot, 12 links, 11 joints
Links:
- link Link1: geometry collision mesh filename=../robot_arm_assets/cr3/meshes/Link1.STL scale=1.00000 1.00000 1.00000; visual mesh filename=../robot_arm_assets/cr3/meshes/Link1.STL scale=1.00000 1.00000 1.00000
- link Link2: geometry collision mesh filename=../robot_arm_assets/cr3/meshes/Link2.STL scale=1.00000 1.00000 1.00000; visual mesh filename=../robot_arm_assets/cr3/meshes/Link2.STL scale=1.00000 1.00000 1.00000
- link Link3: geometry collision mesh filename=../robot_arm_assets/cr3/meshes/Link3.STL scale=1.00000 1.00000 1.00000; visual mesh filename=../robot_arm_assets/cr3/meshes/Link3.STL scale=1.00000 1.00000 1.00000
- link Link4: geometry collision mesh filename=../robot_arm_assets/cr3/meshes/Link4.STL scale=1.00000 1.00000 1.00000; visual mesh filename=../robot_arm_assets/cr3/meshes/Link4.STL scale=1.00000 1.00000 1.00000
- link Link5: geometry collision mesh filename=../robot_arm_assets/cr3/meshes/Link5.STL scale=1.00000 1.00000 1.00000; visual mesh filename=../robot_arm_assets/cr3/meshes/Link5.STL scale=1.00000 1.00000 1.00000
- link Link6: geometry collision mesh filename=../robot_arm_assets/cr3/meshes/Link6.STL scale=1.00000 1.00000 1.00000; visual mesh filename=../robot_arm_assets/cr3/meshes/Link6.STL scale=1.00000 1.00000 1.00000
- link base_link: geometry collision mesh filename=../robot_arm_assets/cr3/meshes/base_link.STL scale=1.00000 1.00000 1.00000; visual mesh filename=../robot_arm_assets/cr3/meshes/base_link.STL scale=1.00000 1.00000 1.00000
- link tactip_body_link: geometry collision mesh filename=../sensor_assets/flat_tactip/../standard_tactip/body/tactip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 scale=1.00000 1.00000 1.00000; visual mesh filename=../sensor_assets/flat_tactip/../standard_tactip/body/tactip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 scale=1.00000 1.00000 1.00000
- link tactip_tip_link: geometry collision mesh filename=../sensor_assets/flat_tactip/tip/skin.obj scale=1.00000 1.00000 1.00000; visual mesh filename=../sensor_assets/flat_tactip/tip/skin.obj scale=1.00000 1.00000 1.00000

File: tactile_sim/assets/embodiment_assets/combined_urdfs/cr3_right_angle_digit.urdf (robot description, URDF)
Before this commit: robot cr3_robot, 12 links, 11 joints
Links:
- link digit_tip_link: geometry collision mesh filename=../sensor_assets/right_angle_digit/../standard_digit/tip/di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 scale=1.05000 1.05000 1.00000; visual mesh filename=../sensor_assets/right_angle_digit/../standard_digit/tip/di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 scale=1.05000 1.05000 1.00000

File: tactile_sim/assets/embodiment_assets/combined_urdfs/cr3_standard_digit.urdf (robot description, URDF)
Before this commit: robot cr3_robot, 12 links, 11 joints
Links:
- link digit_tip_link: geometry collision mesh filename=../sensor_assets/standard_digit/tip/digit_core.stl scale=1.05000 1.05000 1.00000; visual mesh filename=../sensor_assets/standard_digit/tip/digit_skin.stl scale=1.05000 1.05000 1.00000

File: tactile_sim/assets/embodiment_assets/combined_urdfs/cr3_standard_digitac.urdf (robot description, URDF)
Before this commit: robot cr3_robot, 12 links, 11 joints
Links:
- link digitac_tip_link: geometry collision mesh filename=../sensor_assets/standard_digitac/tip/digitac_skin.stl scale=1.00000 1.00000 1.00000; visual mesh filename=../sensor_assets/standard_digitac/tip/digitac_skin.stl scale=1.00000 1.00000 1.00000

File: tactile_sim/assets/embodiment_assets/combined_urdfs/franka_panda_right_angle_digit.urdf (robot description, URDF)
Before this commit: robot panda, 13 links, 12 joints
Links:
- link digit_tip_link: geometry collision mesh filename=../sensor_assets/right_angle_digit/../standard_digit/tip/di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 scale=1.05000 1.05000 1.00000; visual mesh filename=../sensor_assets/right_angle_digit/../standard_digit/tip/di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 scale=1.05000 1.05000 1.00000

File: tactile_sim/assets/embodiment_assets/combined_urdfs/franka_panda_standard_digit.urdf (robot description, URDF)
Before this commit: robot panda, 13 links, 12 joints
Links:
- link digit_tip_link: geometry collision mesh filename=../sensor_assets/standard_digit/tip/digit_core.stl scale=1.05000 1.05000 1.00000; visual mesh filename=../sensor_assets/standard_digit/tip/digit_skin.stl scale=1.05000 1.05000 1.00000

File: tactile_sim/assets/embodiment_assets/combined_urdfs/franka_panda_standard_digitac.urdf (robot description, URDF)
Before this commit: robot panda, 13 links, 12 joints
Links:
- link digitac_tip_link: geometry collision mesh filename=../sensor_assets/standard_digitac/tip/digitac_skin.stl scale=1.00000 1.00000 1.00000; visual mesh filename=../sensor_assets/standard_digitac/tip/digitac_skin.stl scale=1.00000 1.00000 1.00000

File: tactile_sim/assets/embodiment_assets/combined_urdfs/kuka_iiwa_right_angle_digit.urdf (robot description, URDF)
Before this commit: robot lbr_iiwa, 13 links, 12 joints
Links:
- link digit_tip_link: geometry collision mesh filename=../sensor_assets/right_angle_digit/../standard_digit/tip/di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 scale=1.05000 1.05000 1.00000; visual mesh filename=../sensor_assets/right_angle_digit/../standard_digit/tip/di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 scale=1.05000 1.05000 1.00000

File: tactile_sim/assets/embodiment_assets/combined_urdfs/kuka_iiwa_standard_digit.urdf (robot description, URDF)
Before this commit: robot lbr_iiwa, 13 links, 12 joints
Links:
- link digit_tip_link: geometry collision mesh filename=../sensor_assets/standard_digit/tip/digit_core.stl scale=1.05000 1.05000 1.00000; visual mesh filename=../sensor_assets/standard_digit/tip/digit_skin.stl scale=1.05000 1.05000 1.00000

File: tactile_sim/assets/embodiment_assets/combined_urdfs/kuka_iiwa_standard_digitac.urdf (robot description, URDF)
Before this commit: robot lbr_iiwa, 13 links, 12 joints
Links:
- link digitac_tip_link: geometry collision mesh filename=../sensor_assets/standard_digitac/tip/digitac_skin.stl scale=1.00000 1.00000 1.00000; visual mesh filename=../sensor_assets/standard_digitac/tip/digitac_skin.stl scale=1.00000 1.00000 1.00000

File: tactile_sim/assets/embodiment_assets/combined_urdfs/mg400_flat_tactip.urdf (robot description, URDF)
Before this commit: robot mg400, 13 links, 12 joints
Links:
- added link world, mass 0.00000
Joints:
- added joint world_joint: type fixed, parent world, child base_link, origin xyz=0.00000 0.00000 0.00000 rpy=0.00000 -0.00000 -3.14000, axis 0.00000 0.00000 0.00000

File: tactile_sim/assets/embodiment_assets/combined_urdfs/mg400_mini_tactip.urdf (robot description, URDF)
Before this commit: robot mg400, 13 links, 12 joints
Links:
- added link world, mass 0.00000
Joints:
- added joint world_joint: type fixed, parent world, child base_link, origin xyz=0.00000 0.00000 0.00000 rpy=0.00000 -0.00000 -3.14000, axis 0.00000 0.00000 0.00000

File: tactile_sim/assets/embodiment_assets/combined_urdfs/mg400_right_angle_digit.urdf (robot description, URDF)
Before this commit: robot mg400, 13 links, 12 joints
Links:
- added link world, mass 0.00000
- link digit_tip_link: geometry collision mesh filename=../sensor_assets/right_angle_digit/../standard_digit/tip/di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 scale=1.05000 1.05000 1.00000; visual mesh filename=../sensor_assets/right_angle_digit/../standard_digit/tip/di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 scale=1.05000 1.05000 1.00000
Joints:
- added joint world_joint: type fixed, parent world, child base_link, origin xyz=0.00000 0.00000 0.00000 rpy=0.00000 -0.00000 -3.14000, axis 0.00000 0.00000 0.00000
- joint joint_dummy1: origin xyz=0.00000 0.00500 -0.06000 rpy=-1.57080 -1.57080 3.14159 -> xyz=0.00000 0.00500 -0.06000 rpy=-1.57080 -1.57080 1.57080

File: tactile_sim/assets/embodiment_assets/combined_urdfs/mg400_right_angle_digitac.urdf (robot description, URDF)
Before this commit: robot mg400, 13 links, 12 joints
Links:
- added link world, mass 0.00000
Joints:
- added joint world_joint: type fixed, parent world, child base_link, origin xyz=0.00000 0.00000 0.00000 rpy=0.00000 -0.00000 -3.14000, axis 0.00000 0.00000 0.00000
- joint joint_dummy1: origin xyz=0.00000 0.00500 -0.06000 rpy=-1.57080 -1.57080 3.14159 -> xyz=0.00000 0.00500 -0.06000 rpy=-1.57080 -1.57080 1.57080

File: tactile_sim/assets/embodiment_assets/combined_urdfs/mg400_right_angle_tactip.urdf (robot description, URDF)
Before this commit: robot mg400, 14 links, 13 joints
Links:
- added link world, mass 0.00000
Joints:
- added joint world_joint: type fixed, parent world, child base_link, origin xyz=0.00000 0.00000 0.00000 rpy=0.00000 -0.00000 -3.14000, axis 0.00000 0.00000 0.00000
- joint joint_dummy1: origin xyz=0.00000 0.00500 -0.06000 rpy=-1.57080 -1.57080 3.14159 -> xyz=0.00000 0.00500 -0.06000 rpy=-1.57080 -1.57080 1.57080

File: tactile_sim/assets/embodiment_assets/combined_urdfs/mg400_standard_digit.urdf (robot description, URDF)
Before this commit: robot mg400, 13 links, 12 joints
Links:
- added link world, mass 0.00000
- link digit_tip_link: geometry collision mesh filename=../sensor_assets/standard_digit/tip/digit_core.stl scale=1.05000 1.05000 1.00000; visual mesh filename=../sensor_assets/standard_digit/tip/digit_skin.stl scale=1.05000 1.05000 1.00000
Joints:
- added joint world_joint: type fixed, parent world, child base_link, origin xyz=0.00000 0.00000 0.00000 rpy=0.00000 -0.00000 -3.14000, axis 0.00000 0.00000 0.00000

File: tactile_sim/assets/embodiment_assets/combined_urdfs/mg400_standard_digitac.urdf (robot description, URDF)
Before this commit: robot mg400, 13 links, 12 joints
Links:
- added link world, mass 0.00000
- link digitac_tip_link: geometry collision mesh filename=../sensor_assets/standard_digitac/tip/digitac_skin.stl scale=1.00000 1.00000 1.00000; visual mesh filename=../sensor_assets/standard_digitac/tip/digitac_skin.stl scale=1.00000 1.00000 1.00000
Joints:
- added joint world_joint: type fixed, parent world, child base_link, origin xyz=0.00000 0.00000 0.00000 rpy=0.00000 -0.00000 -3.14000, axis 0.00000 0.00000 0.00000

File: tactile_sim/assets/embodiment_assets/combined_urdfs/mg400_standard_tactip.urdf (robot description, URDF)
Before this commit: robot mg400, 13 links, 12 joints
Links:
- added link world, mass 0.00000
Joints:
- added joint world_joint: type fixed, parent world, child base_link, origin xyz=0.00000 0.00000 0.00000 rpy=0.00000 -0.00000 -3.14000, axis 0.00000 0.00000 0.00000

File: tactile_sim/assets/embodiment_assets/combined_urdfs/ur5_right_angle_digit.urdf (robot description, URDF)
Before this commit: robot universal_robot, 12 links, 11 joints
Links:
- link digit_tip_link: geometry collision mesh filename=../sensor_assets/right_angle_digit/../standard_digit/tip/di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 scale=1.05000 1.05000 1.00000; visual mesh filename=../sensor_assets/right_angle_digit/../standard_digit/tip/di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 scale=1.05000 1.05000 1.00000

File: tactile_sim/assets/embodiment_assets/combined_urdfs/ur5_standard_digit.urdf (robot description, URDF)
Before this commit: robot universal_robot, 12 links, 11 joints
Links:
- link digit_tip_link: geometry collision mesh filename=../sensor_assets/standard_digit/tip/digit_core.stl scale=1.05000 1.05000 1.00000; visual mesh filename=../sensor_assets/standard_digit/tip/digit_skin.stl scale=1.05000 1.05000 1.00000
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
Commit message: update flat_tactip core

File: tactile_sim/assets/embodiment_assets/combined_urdfs/cr3_flat_tactip.urdf (robot description, URDF)
Before this commit: robot cr3_robot, 12 links, 11 joints
Links:
- link tactip_tip_link: geometry collision mesh filename=../sensor_assets/flat_tactip/tip/core.obj scale=1.00000 1.00000 1.00000; visual mesh filename=../sensor_assets/flat_tactip/tip/skin.obj scale=1.00000 1.00000 1.00000

File: tactile_sim/assets/embodiment_assets/combined_urdfs/franka_panda_flat_tactip.urdf (robot description, URDF)
Before this commit: robot panda, 13 links, 12 joints
Links:
- link tactip_tip_link: geometry collision mesh filename=../sensor_assets/flat_tactip/tip/core.obj scale=1.00000 1.00000 1.00000; visual mesh filename=../sensor_assets/flat_tactip/tip/skin.obj scale=1.00000 1.00000 1.00000

File: tactile_sim/assets/embodiment_assets/combined_urdfs/kuka_iiwa_flat_tactip.urdf (robot description, URDF)
Before this commit: robot lbr_iiwa, 13 links, 12 joints
Links:
- link tactip_tip_link: geometry collision mesh filename=../sensor_assets/flat_tactip/tip/core.obj scale=1.00000 1.00000 1.00000; visual mesh filename=../sensor_assets/flat_tactip/tip/skin.obj scale=1.00000 1.00000 1.00000

File: tactile_sim/assets/embodiment_assets/combined_urdfs/mg400_flat_tactip.urdf (robot description, URDF)
Before this commit: robot mg400, 14 links, 13 joints
Links:
- link tactip_tip_link: geometry collision mesh filename=../sensor_assets/flat_tactip/tip/core.obj scale=1.00000 1.00000 1.00000; visual mesh filename=../sensor_assets/flat_tactip/tip/skin.obj scale=1.00000 1.00000 1.00000

File: tactile_sim/assets/embodiment_assets/combined_urdfs/ur5_flat_tactip.urdf (robot description, URDF)
Before this commit: robot universal_robot, 12 links, 11 joints
Links:
- link tactip_tip_link: geometry collision mesh filename=../sensor_assets/flat_tactip/tip/core.obj scale=1.00000 1.00000 1.00000; visual mesh filename=../sensor_assets/flat_tactip/tip/skin.obj scale=1.00000 1.00000 1.00000

File: tactile_sim/assets/sensor_assets/flat_tactip/flat_tactip.urdf (robot description, URDF)
Before this commit: robot universal_robot, 3 links, 2 joints
Links:
- link tactip_tip_link: geometry collision mesh filename=tip/core.obj scale=1.0 1.0 1.0; visual mesh filename=tip/skin.obj scale=1.0 1.0 1.0
